File: Motion Detector.sch (KiCad schematic (older format))
At the start: 12 parts, among them J1 Jack-DC, J2 Conn_01x03, J3 Conn_01x03, Q1 BC547, Q2 BC547, U1 NodeMCU_1.0_(ESP-12E)

Commit message: pcb file completed
Parts:
- C1, C2: symbol Device:C -> Motion_Detector:Device_C
- D1: symbol Device:D -> Motion_Detector:Device_D
- J1: footprint Connector:JWT_A3963_1x02_P3.96mm_Vertical -> Connector_BarrelJack:Connector_Barrel_2pole; symbol Connector:Jack-DC -> Motion_Detector:Connector_Jack-DC
- J2, J3: symbol Connector_Generic:Conn_01x03 -> Motion_Detector:Connector_Generic_Conn_01x03
- Q1, Q2: symbol Transistor_BJT:BC547 -> Motion_Detector:Transistor_BJT_BC547
- R1, R2, R3: symbol Device:R -> Motion_Detector:Device_R
- U1: footprint ESP8266:NodeMCU1.0(12-E) -> ESP8266:NodeMCU_1.0_small; symbol ESP8266:NodeMCU_1.0_(ESP-12E) -> Motion_Detector:ESP8266_NodeMCU_1.0_(ESP-12E)
Connections:
- net DB1: now also R2.2
- net DB2: now also R1.2
Changed lines of the file:
@@
 EESchema Schematic File Version 4
+LIBS:Motion Detector-cache
 EELAYER 26 0
 EELAYER END
@@
 $EndDescr
 $Comp
-L ESP8266:NodeMCU_1.0_(ESP-12E) U1
+L Motion_Detector:ESP8266_NodeMCU_1.0_(ESP-12E) U1
 U 1 1 5C03AC3F
 P 5200 3800
 F 0 "U1" H 5200 4650 60  0000 C CNN
 F 1 "NodeMCU_1.0_(ESP-12E)" H 5200 2950 60  0000 C CNN
-F 2 "ESP8266:NodeMCU1.0(12-E)" H 4600 2950 60  0001 C CNN
+F 2 "ESP8266:NodeMCU_1.0_small" H 4600 2950 60  0001 C CNN
 F 3 "" H 4600 2950 60  0000 C CNN
 	1    5200 3800
@@
 $EndComp
 $Comp
-L Connector_Generic:Conn_01x03 J2
+L Motion_Detector:Connector_Generic_Conn_01x03 J2
 U 1 1 5C03BA21
 P 2400 5100
@@
 $EndComp
 $Comp
-L Connector_Generic:Conn_01x03 J3
+L Motion_Detector:Connector_Generic_Conn_01x03 J3
 U 1 1 5C03BA44
 P 2400 5800
@@
 $EndComp
 $Comp
-L Connector:Jack-DC J1
+L Motion_Detector:Connector_Jack-DC J1
 U 1 1 5C03BA65
 P 2000 3600
 F 0 "J1" H 2000 3810 50  0000 C CNN
 F 1 "Jack-DC" H 2000 3425 50  0000 C CNN
-F 2 "Connector:JWT_A3963_1x02_P3.96mm_Vertical" H 2050 3560 50  0001 C CNN
+F 2 "Connector_BarrelJack:Connector_Barrel_2pole" H 2050 3560 50  0001 C CNN
 F 3 "" H 2050 3560 50  0001 C CNN
 	1    2000 3600
@@
 $EndComp
 $Comp
-L Transistor_BJT:BC547 Q1
+L Motion_Detector:Transistor_BJT_BC547 Q1
 U 1 1 5C03C05C
 P 3750 5100
@@
 $EndComp
 $Comp
-L Device:C C1
+L Motion_Detector:Device_C C1
 U 1 1 5C03C0BF
 P 3150 5100
@@
 $EndComp
 $Comp
-L Device:R R3
+L Motion_Detector:Device_R R3
 U 1 1 5C03C0EC
 P 5300 5150
@@
 $EndComp
 $Comp
-L Device:R R1
+L Motion_Detector:Device_R R1
 U 1 1 5C03CBC5
 P 3500 4950
@@
 $EndComp
 $Comp
-L power:GND #PWR01
+L Motion_Detector:power_GND #PWR01
 U 1 1 5C03CC70
 P 4050 4800
 F 0 "#PWR01" H 4050 4550 50  0001 C CNN
-F 1 "GND" H 4050 4650 50  0000 C CNN
+F 1 "power_GND" H 4050 4650 50  0000 C CNN
 F 2 "" H 4050 4800 50  0001 C CNN
 F 3 "" H 4050 4800 50  0001 C CNN
@@
 $EndComp
 $Comp
-L Device:D D1
+L Motion_Detector:Device_D D1
 U 1 1 5C03D060
 P 5750 5150
@@
 $EndComp
 $Comp
-L Transistor_BJT:BC547 Q2
+L Motion_Detector:Transistor_BJT_BC547 Q2
 U 1 1 5C03DC7C
 P 3750 5800
@@
 $EndComp
 $Comp
-L Device:C C2
+L Motion_Detector:Device_C C2
 U 1 1 5C03DC82
 P 3150 5800
@@
 $EndComp
 $Comp
-L Device:R R2
+L Motion_Detector:Device_R R2
 U 1 1 5C03DC8A
 P 3500 5650
@@
 $EndComp
 $Comp
-L power:GND #PWR02
+L Motion_Detector:power_GND #PWR02
 U 1 1 5C03DC92
 P 4050 5500
 F 0 "#PWR02" H 4050 5250 50  0001 C CNN
-F 1 "GND" H 4050 5350 50  0000 C CNN
+F 1 "power_GND" H 4050 5350 50  0000 C CNN
 F 2 "" H 4050 5500 50  0001 C CNN
 F 3 "" H 4050 5500 50  0001 C CNN
@@
 $EndComp
 $Comp
-L power:GND #PWR03
+L Motion_Detector:power_GND #PWR03
 U 1 1 5C03DE7B
 P 4150 3200
 F 0 "#PWR03" H 4150 2950 50  0001 C CNN
-F 1 "GND" H 4150 3050 50  0000 C CNN
+F 1 "power_GND" H 4150 3050 50  0000 C CNN
 F 2 "" H 4150 3200 50  0001 C CNN
 F 3 "" H 4150 3200 50  0001 C CNN
@@
 $EndComp
 $Comp
-L power:GND #PWR04
+L Motion_Detector:power_GND #PWR04
 U 1 1 5C03DEAA
 P 4000 3900
 F 0 "#PWR04" H 4000 3650 50  0001 C CNN
-F 1 "GND" H 4000 3750 50  0000 C CNN
+F 1 "power_GND" H 4000 3750 50  0000 C CNN
 F 2 "" H 4000 3900 50  0001 C CNN
 F 3 "" H 4000 3900 50  0001 C CNN
@@
 $EndComp
 $Comp
-L power:GND #PWR05
+L Motion_Detector:power_GND #PWR05
 U 1 1 5C03DF90
 P 6150 3600
 F 0 "#PWR05" H 6150 3350 50  0001 C CNN
-F 1 "GND" H 6150 3450 50  0000 C CNN
+F 1 "power_GND" H 6150 3450 50  0000 C CNN
 F 2 "" H 6150 3600 50  0001 C CNN
 F 3 "" H 6150 3600 50  0001 C CNN
@@
 $EndComp
 $Comp
-L power:GND #PWR06
+L Motion_Detector:power_GND #PWR06
 U 1 1 5C03E077
 P 6450 3200
 F 0 "#PWR06" H 6450 2950 50  0001 C CNN
-F 1 "GND" H 6450 3050 50  0000 C CNN
+F 1 "power_GND" H 6450 3050 50  0000 C CNN
 F 2 "" H 6450 3200 50  0001 C CNN
 F 3 "" H 6450 3200 50  0001 C CNN
@@
 $EndComp
 $Comp
-L power:GND #PWR07
+L Motion_Detector:power_GND #PWR07
 U 1 1 5C03E348
 P 2750 5200
 F 0 "#PWR07" H 2750 4950 50  0001 C CNN
-F 1 "GND" H 2750 5050 50  0000 C CNN
+F 1 "power_GND" H 2750 5050 50  0000 C CNN
 F 2 "" H 2750 5200 50  0001 C CNN
 F 3 "" H 2750 5200 50  0001 C CNN
@@
 $EndComp
 $Comp
-L power:GND #PWR08
+L Motion_Detector:power_GND #PWR08
 U 1 1 5C03E377
 P 2750 5900
 F 0 "#PWR08" H 2750 5650 50  0001 C CNN
-F 1 "GND" H 2750 5750 50  0000 C CNN
+F 1 "power_GND" H 2750 5750 50  0000 C CNN
 F 2 "" H 2750 5900 50  0001 C CNN
 F 3 "" H 2750 5900 50  0001 C CNN
@@
 $EndComp
 $Comp
-L power:GND #PWR09
+L Motion_Detector:power_GND #PWR09
 U 1 1 5C03E3A6
 P 2500 3700
 F 0 "#PWR09" H 2500 3450 50  0001 C CNN
-F 1 "GND" H 2500 3550 50  0000 C CNN
+F 1 "power_GND" H 2500 3550 50  0000 C CNN
 F 2 "" H 2500 3700 50  0001 C CNN
 F 3 "" H 2500 3700 50  0001 C CNN
@@
 $EndComp
 $Comp
-L power:VCC #PWR010
+L Motion_Detector:power_VCC #PWR010
 U 1 1 5C03E801
 P 2500 3500
 F 0 "#PWR010" H 2500 3350 50  0001 C CNN
-F 1 "VCC" H 2500 3650 50  0000 C CNN
+F 1 "power_VCC" H 2500 3650 50  0000 C CNN
 F 2 "" H 2500 3500 50  0001 C CNN
 F 3 "" H 2500 3500 50  0001 C CNN
@@
 $EndComp
 $Comp
-L power:VCC #PWR011
+L Motion_Detector:power_VCC #PWR011
 U 1 1 5C03E8C7
 P 6450 3100
 F 0 "#PWR011" H 6450 2950 50  0001 C CNN
-F 1 "VCC" H 6450 3250 50  0000 C CNN
+F 1 "power_VCC" H 6450 3250 50  0000 C CNN
 F 2 "" H 6450 3100 50  0001 C CNN
 F 3 "" H 6450 3100 50  0001 C CNN
@@
 $EndComp
 $Comp
-L power:VCC #PWR012
+L Motion_Detector:power_VCC #PWR012
 U 1 1 5C03E932
 P 2750 5000
 F 0 "#PWR012" H 2750 4850 50  0001 C CNN
-F 1 "VCC" H 2750 5150 50  0000 C CNN
+F 1 "power_VCC" H 2750 5150 50  0000 C CNN
 F 2 "" H 2750 5000 50  0001 C CNN
 F 3 "" H 2750 5000 50  0001 C CNN
@@
 $EndComp
 $Comp
-L power:VCC #PWR013
+L Motion_Detector:power_VCC #PWR013
 U 1 1 5C03EA39
 P 2750 5700
 F 0 "#PWR013" H 2750 5550 50  0001 C CNN
-F 1 "VCC" H 2750 5850 50  0000 C CNN
+F 1 "power_VCC" H 2750 5850 50  0000 C CNN
 F 2 "" H 2750 5700 50  0001 C CNN
 F 3 "" H 2750 5700 50  0001 C CNN
@@
 $EndComp
 $Comp
-L power:+3.3V #PWR014
+L Motion_Detector:power_+3.3V #PWR014
 U 1 1 5C03ECCE
 P 4150 3100
 F 0 "#PWR014" H 4150 2950 50  0001 C CNN
-F 1 "+3.3V" H 4150 3240 50  0000 C CNN
+F 1 "power_+3.3V" H 4150 3240 50  0000 C CNN
 F 2 "" H 4150 3100 50  0001 C CNN
 F 3 "" H 4150 3100 50  0001 C CNN
@@
 $EndComp
 $Comp
-L power:+3.3V #PWR015
+L Motion_Detector:+3.3V #PWR015
 U 1 1 5C03ED10
 P 4000 4000
@@
 $EndComp
 $Comp
-L power:+3.3V #PWR016
+L Motion_Detector:+3.3V #PWR016
 U 1 1 5C03EDD8
 P 6150 3500
@@
 	4200 4000 4400 4000
 Wire Wire Line
-	3300 5100 3550 5100
-Wire Wire Line
-	3300 5800 3550 5800
+	3300 5100 3500 5100
+Connection ~ 3500 5100
+Wire Wire Line
+	3500 5100 3550 5100
+Wire Wire Line
+	3300 5800 3500 5800
+Connection ~ 3500 5800
+Wire Wire Line
+	3500 5800 3550 5800
 $EndSCHEMATC
